File: hardware/smartwatch/smartwatch.sch (EAGLE design)
At the start: 40 parts, among them Q5.1 DMP1045U, U2 HM-11, U4 MCP1700T-3302E/TT, U5 MCP73832, U6 MAX17043, U7 KSSG33J12, X1.1 FC-135

Commit message: redid brd
Parts:
- added BTN1, BTN2, BTN3, BTN4: SPST.B3U-3000P(M), omron:SPST.B3U-3000P(M)
- added R5.3, R5.4: 47K, resistor:R-EU_R2012
- added R8.1, R8.2, R8.3, R8.4: 39R, resistor:R-EU_R2012
Connections:
- net N$6 renamed VDDCORE
- new net BUT1: R8.1.1, U1.PA02/EI2/AD0/Y0/VOUT
- new net BUT2: R8.2.1, U1.CLK0/EI15/PA27
- new net BUT3: R8.3.1, U1.PA14/EI14/XIN/S2P2/S4P2/T3W0/CLK0
- new net BUT4: R8.4.1, U1.PA15/EI15/XOUT/S2P3/S4P3/T3W1/CLK1
- new net MBAT: R5.3.2, R5.4.1, U1.PA03/EI3/AD1/Y1/VREFA
- new net N$16: BTN2.1, R8.2.2
- new net N$18: BTN3.1, R8.3.2
- new net N$19: BTN4.1, R8.4.2
- new net N$9: BTN1.1, R8.1.2
- new net PIO0: U1.CLK7/T4W1/S5P1/S3P1/X11/EI7/PA23, U2.PIO0
- net GND: now also BTN1.2, BTN2.2, BTN3.2, BTN4.2, R5.4.2
- net PIO2: now also U1.T5W0/S5P2/S3P2/EI12/PA24; no longer U1.CLK7/T4W1/S5P1/S3P1/X11/EI7/PA23
- net PIO3: now also U1.T5W1/S5P3/S3P3/EI13/PA25; no longer U1.T5W0/S5P2/S3P2/EI12/PA24
- net SCL: no longer U1.PA05/EI5/AD5/AC1/Y3/S0P1/T0W1
- net SDA: no longer U1.PA04/EI4/AD4/AC0/Y2/S0P0/T0W0/VREFB
- net VBAT: now also R5.3.1
Other:
- moved on the sheet: C1.1, C1.2, C1.3, D7.2, JP3, Q7.1, R7.1, U1, U7, X1.1
